Commit message: Add dual GPS navigation stack and sim steering fix

File: src/navegacion_gps/models/cuatri_2gps.urdf (robot description, URDF)
Before this commit: robot quad_ackermann_viewer_safe, 13 links, 12 joints
Links:
- removed link gps1_link
- removed link gps2_link
- added link gps_link2, mass 0.05; collision box size=0.074 0.074 0.015; visual box size=0.07 0.04 0.035
- link front_left_wheel_link: geometry collision cylinder length=0.16 radius=0.24; visual box size=0.24 0.018 0.018
- link front_right_wheel_link: geometry collision cylinder length=0.16 radius=0.24; visual box size=0.24 0.018 0.018
- link rear_left_wheel_link: geometry collision cylinder length=0.16 radius=0.24; visual box size=0.24 0.018 0.018
- link rear_right_wheel_link: geometry collision cylinder length=0.16 radius=0.24; visual box size=0.24 0.018 0.018
Joints:
- removed joint gps1_joint
- removed joint gps2_joint
- added joint gps_joint2: type fixed, parent base_link, child gps_link2, origin xyz=1.00 -0.25 0.62 rpy=0 0 0
- joint gps_joint: origin xyz=0.76 0.04 0.62 rpy=0 0 0 -> xyz=1.00 0.25 0.62 rpy=0 0 0
