Commit message: Pagina terminada y YOLO sin RTSP

File: src/navegacion_gps/models/cuatri_real.urdf (robot description, URDF)
Before this commit: robot quad_ackermann_viewer_safe, 11 links, 10 joints
Links:
- added link gps1_link, mass 0.05; visual box size=0.07 0.04 0.035
- added link gps2_link, mass 0.05; visual box size=0.07 0.04 0.035
Joints:
- added joint gps1_joint: type fixed, parent base_link, child gps1_link, origin xyz=0.94 0.0 0.65 rpy=0 0 0
- added joint gps2_joint: type fixed, parent base_link, child gps2_link, origin xyz=0.0 0.0 0.65 rpy=0 0 0
- joint front_left_wheel_joint: limit lower=-1000 upper=1000 effort=200 velocity=100 -> effort=200 velocity=100; type revolute -> continuous
- joint front_right_wheel_joint: limit lower=-1000 upper=1000 effort=200 velocity=100 -> effort=200 velocity=100; type revolute -> continuous
- joint rear_left_wheel_joint: limit lower=-1000 upper=1000 effort=200 velocity=100 -> effort=200 velocity=100; type revolute -> continuous
- joint rear_right_wheel_joint: limit lower=-1000 upper=1000 effort=200 velocity=100 -> effort=200 velocity=100; type revolute -> continuous
