Commit message: posible sim: corrige drift grid odom

File: src/navegacion_gps/models/cuatri.urdf (robot description, URDF)
Before this commit: robot quad_ackermann_viewer_safe, 11 links, 10 joints
Joints:
- joint front_left_wheel_joint: limit lower=-1000 upper=1000 effort=200 velocity=100 -> effort=200 velocity=100; type revolute -> continuous
- joint front_right_wheel_joint: limit lower=-1000 upper=1000 effort=200 velocity=100 -> effort=200 velocity=100; type revolute -> continuous
- joint rear_left_wheel_joint: limit lower=-1000 upper=1000 effort=200 velocity=100 -> effort=200 velocity=100; type revolute -> continuous
- joint rear_right_wheel_joint: limit lower=-1000 upper=1000 effort=200 velocity=100 -> effort=200 velocity=100; type revolute -> continuous

File: src/navegacion_gps/models/cuatri_real.urdf (robot description, URDF)
Before this commit: robot quad_ackermann_viewer_safe, 13 links, 12 joints
Links:
- removed link gps1_link
- removed link gps2_link
Joints:
- removed joint gps1_joint
- removed joint gps2_joint

File: src/navegacion_gps/models/cuatri_ultrasound.urdf (robot description, URDF)
Before this commit: robot quad_ackermann_viewer_safe, 16 links, 15 joints
Joints:
- joint front_left_wheel_joint: limit lower=-1000 upper=1000 effort=200 velocity=100 -> effort=200 velocity=100; type revolute -> continuous
- joint front_right_wheel_joint: limit lower=-1000 upper=1000 effort=200 velocity=100 -> effort=200 velocity=100; type revolute -> continuous
- joint rear_left_wheel_joint: limit lower=-1000 upper=1000 effort=200 velocity=100 -> effort=200 velocity=100; type revolute -> continuous
- joint rear_right_wheel_joint: limit lower=-1000 upper=1000 effort=200 velocity=100 -> effort=200 velocity=100; type revolute -> continuous
